File: board/board.kicad_pcb (KiCad board)
At the start: 2 copper layers, 21 x 13 mm, 1 part

Commit message: initial
Parts:
- removed LOGO1: Logo_Open_Hardware_Small, Symbol:OSHW-Symbol_6.7x6mm_SilkScreen
- added C1: 100n, Capacitor_SMD:C_0603_1608Metric, F.Cu at (79.9, 93.7)
- added C10: 22uF, Capacitor_SMD:C_0805_2012Metric, F.Cu at (107.2, 96.6)
- added C11: 220u, Capacitor_Tantalum_SMD:CP_EIA-7343-31_Kemet-D, F.Cu at (110.8, 95.8)
- added C12: 1nF, Capacitor_SMD:C_1806_4516Metric, F.Cu at (100.0, 101.1)
- added C2: 100n, Capacitor_SMD:C_0603_1608Metric, F.Cu at (91.7, 95.3)
- added C3: 2.2uF, Capacitor_SMD:C_1210_3225Metric, F.Cu at (78.8, 88.4)
- added C4: 10nF, Capacitor_SMD:C_0603_1608Metric, F.Cu at (90.8, 88.1)
- added C5: 2.2uF, Capacitor_SMD:C_1210_3225Metric, F.Cu at (82.0, 88.4)
- added C6: 2.2uF, Capacitor_SMD:C_1210_3225Metric, F.Cu at (85.2, 88.4)
- added C7: 2.2uF, Capacitor_SMD:C_1210_3225Metric, F.Cu at (88.4, 88.4)
- added C8: 10n, Capacitor_SMD:C_0603_1608Metric, F.Cu at (108.0, 88.2)
- added C9: 22uF, Capacitor_SMD:C_0805_2012Metric, F.Cu at (107.2, 93.0)
- added D1: BAV21WS-HE3-18, Diode_SMD:D_SOD-323_HandSoldering, F.Cu at (91.9, 91.7)
- added D2: 1N4148, Diode_SMD:D_SOD-323_HandSoldering, F.Cu at (86.4, 100.2)
- added D3: CUS15S30,H3F, Diode_SMD:D_SOD-323_HandSoldering, F.Cu at (108.7, 90.0)
- added J1: 013_PoE_rectified, on_edge:on_edge_2x05_device, F.Cu at (77.0, 80.6)
- added J2: 003_power, on_edge:on_edge_2x05_host, F.Cu at (114.0, 80.5)
- added R1: 100k, Resistor_SMD:R_0603_1608Metric, F.Cu at (88.2, 99.7)
- added R2: 20k, Resistor_SMD:R_0603_1608Metric, F.Cu at (89.7, 99.7)
- added R3: 41.2R, Resistor_SMD:R_0603_1608Metric, F.Cu at (81.5, 93.7)
- added R4: 24.9k, Resistor_SMD:R_0603_1608Metric, F.Cu at (83.7, 99.9)
- added R5: 52.3k, Resistor_SMD:R_0603_1608Metric, F.Cu at (91.2, 99.7)
- added R6: 10k, Resistor_SMD:R_0603_1608Metric, F.Cu at (92.3, 88.0)
- added R7: 5k, Resistor_SMD:R_0603_1608Metric, F.Cu at (88.9, 102.0)
- added R8: 20R, Resistor_SMD:R_0603_1608Metric, F.Cu at (111.1, 88.2)
- added U1: MP8007, Package_DFN_QFN:QFN-28-1EP_4x5mm_P0.5mm_EP2.65x3.65mm_ThermalVias, F.Cu at (87.2, 93.8)
- added U2: POE30P-50L, b033:Transformer_Coilcraft_POE30P, F.Cu at (99.7, 93.2)
Routing:
- net GND: track 0.00 -> 68.3 mm, vias 0 -> 34
- net /Controller/GNDPWR: track 0.00 -> 57.2 mm, vias 0 -> 1
- net /Controller/PoE+: track 0.00 -> 56.3 mm, vias 0 -> 5
- net /Controller/5V: track 0.00 -> 51.6 mm, vias 0 -> 1
- net Net-(J2-Pad9): track 0.00 -> 32.2 mm
- net /Controller/PoE-: track 0.00 -> 21.3 mm, vias 0 -> 2
- net Net-(D2-Pad2): track 0.00 -> 17.6 mm
- net Net-(C2-Pad1): track 0.00 -> 16.5 mm
- net Net-(C8-Pad1): track 0.00 -> 6.92 mm
- net Net-(D1-Pad2): track 0.00 -> 6.47 mm
- net Net-(R1-Pad2): track 0.00 -> 4.75 mm
- net Net-(R4-Pad2): track 0.00 -> 4.31 mm
- net Net-(R5-Pad1): track 0.00 -> 4.08 mm
- net Net-(R3-Pad1): track 0.00 -> 3.46 mm
- net Net-(C4-Pad1): track 0.00 -> 3.23 mm
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- added copper zone on B.Cu, net /Controller/GNDPWR
- added copper zone on F.Cu, net /Controller/GNDPWR
- added copper zone on F.Cu, net /Controller/PoE+
- added copper zone on B.Cu, net GND
- added copper zone on F.Cu, net GND
Other:
- board size 21 x 13 mm -> 37 x 29 mm
- rule pad_to_mask_clearance: 0 -> 0.04
- board text added: "osf.b033.v1.0"
